File: hardware/RC-Multiswitch-ESP32-C3-NEG.kicad_sch (KiCad schematic)
At the start: 31 parts, among them CN1 UART A, CN2 5-12V, J1 Ausgaenge, J5 UART B, U1 ESP32-C3 SuperMini, U2 ULN2803A

Commit message: Hardware: TBD62083APG statt ULN2803A, Original-Projekt entfernt
ULN2803A ist abgekuendigt. Der TBD62083APG (DMOS) hat dieselbe Pinbelegung und passt in denselben Sockel, Leiterbahnen und Netze bleiben unveraendert. Schaltplan-Symbol, Bauteilwert, Bestueckungsdruck und Doku angepasst.

Co-Authored-By: Claude Opus 5.5 <noreply@anthropic.com>
Claude-Session: https://claude.ai/code/session_0118D4qppRkb6gR5m3R2CZyV
Parts:
- U2: value ULN2803A -> TBD62083APG; symbol Transistor_Array:ULN2803A -> local:TBD62083APG
Other:
- note added: "ESP32-C3 SuperMini Multiswitch: 8 Kanaele (TBD62083APG) + CRSF - Entwurf v0.3"
- note removed: "ESP32-C3 SuperMini Multiswitch: 8 Kanaele (ULN2803A) + CRSF - Entwurf v0.3"
- title: RC Multiswitch ESP32-C3 SuperMini (ULN2803A, negativ schaltend) -> RC Multiswitch ESP32-C3 SuperMini (TBD62083APG, negativ schaltend)
Changed lines of the file:
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@@
 	(paper "A4")
 	(title_block
-		(title "RC Multiswitch ESP32-C3 SuperMini (ULN2803A, negativ schaltend)")
+		(title "RC Multiswitch ESP32-C3 SuperMini (TBD62083APG, negativ schaltend)")
 		(date "2026-10-14")
 		(rev "v0.3")
@@
 		)
 	)
-	(text "ESP32-C3 SuperMini Multiswitch: 8 Kanaele (ULN2803A) + CRSF  -  Entwurf v0.3"
+	(text "ESP32-C3 SuperMini Multiswitch: 8 Kanaele (TBD62083APG) + CRSF  -  Entwurf v0.3"
 		(exclude_from_sim no)
 		(at 15 14 0)
@@
 	)
 	(symbol
-		(lib_id "Transistor_Array:ULN2803A")
+		(lib_id "local:TBD62083APG")
 		(at 165.1 101.6 0)
 		(unit 1)
@@
 			)
 		)
-		(property "Value" "ULN2803A"
+		(property "Value" "TBD62083APG"
 			(at 165.1 122.88 0)
 			(effects
